File: UV_LED_Driver_Combined/UV_LED_Driver.kicad_pcb (KiCad board)
At the start: 2 copper layers, 52.7 x 165.1 mm, 34 parts, among them J1 Barrel_Jack, J2 Conn_01x05, Q1 IPP80N03S4L-03, Q2 IPP80N03S4L-03, Q3 IPP80N03S4L-03, Q4 IPP80N03S4L-03, Q5 IPP80N03S4L-03, SW1 SW_SPST, U1 STM32L011D4Px, U2 LP3992-33B5F

Commit message: Changed TO225 NPN (MJE340) to SOT223 NPN (PZT2222A)
Parts:
- D1, D2, D3, D4, D5: value LED_Connector -> LED_Series
- moved R16 83.8 mm to (54.6, 41.9)
- moved R14 83.8 mm to (62.2, 55.9)
- moved R15 83.8 mm to (62.2, 52.1)
- moved R4 27.9 mm to (62.2, 111.8)
- moved R6 27.9 mm to (54.6, 97.8)
- moved R2 27.9 mm to (62.2, 80.0)
- moved D4 27.9 mm to (78.7, 142.2)
- moved D5 27.9 mm to (78.7, 170.2)
- moved Q4 27.9 mm to (54.6, 139.7)
- moved Q5 27.9 mm to (54.6, 167.6)
- moved R3 27.9 mm to (54.6, 69.8)
- moved R5 27.9 mm to (62.2, 108.0)
- moved R9 27.9 mm to (54.6, 125.7)
- moved R1 27.9 mm to (62.2, 83.8)
- moved R7 27.9 mm to (62.2, 139.7)
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Connections:
- net /LED_Controller/3V3 renamed /LED_Controller_Module/3V3
- net /LED_Controller/LED_ADC renamed /LED_Controller_Module/LED_ADC
- net /LED_Controller/LID_SW renamed /LED_Controller_Module/LID_SW
- net /LED_Controller/NRST renamed /LED_Controller_Module/NRST
- net /LED_Controller/SWCLK renamed /LED_Controller_Module/SWCLK
- net /LED_Controller/SWDIO renamed /LED_Controller_Module/SWDIO
- net Net-(D1-Pad1) renamed /UV_LED_Driver_Module1/LED_CATHODE_OUT
- net Net-(D2-Pad1) renamed /UV_LED_Driver_Module2/LED_CATHODE_OUT
- net Net-(D3-Pad1) renamed /UV_LED_Driver_Module3/LED_CATHODE_OUT
- net Net-(D4-Pad1) renamed /UV_LED_Driver_Module4/LED_CATHODE_OUT
- net Net-(D5-Pad1) renamed /STD_LED_Driver_Module/LED_CATHODE_OUT
- R1 pad 1: Net-(Q1-Pad1) -> Net-(Q2-Pad1)
- R10 pad 1: Net-(Q4-Pad1) -> Net-(Q5-Pad1)
- R11 pad 2: Net-(Q4-Pad1) -> Net-(Q5-Pad1)
- R12 pad 1: Net-(Q4-Pad3) -> Net-(Q5-Pad3)
- R14 pad 1: Net-(Q5-Pad1) -> Net-(Q1-Pad1)
- R15 pad 2: Net-(Q5-Pad1) -> Net-(Q1-Pad1)
- R16 pad 1: Net-(Q5-Pad3) -> Net-(Q1-Pad3)
- R2 pad 2: Net-(Q1-Pad1) -> Net-(Q2-Pad1)
- R3 pad 1: Net-(Q1-Pad3) -> Net-(Q2-Pad3)
- R4 pad 1: Net-(Q2-Pad1) -> Net-(Q3-Pad1)
- R5 pad 2: Net-(Q2-Pad1) -> Net-(Q3-Pad1)
- R6 pad 1: Net-(Q2-Pad3) -> Net-(Q3-Pad3)
- R7 pad 1: Net-(Q3-Pad1) -> Net-(Q4-Pad1)
- R8 pad 2: Net-(Q3-Pad1) -> Net-(Q4-Pad1)
- R9 pad 1: Net-(Q3-Pad3) -> Net-(Q4-Pad3)
