File: UV_LED_Driver_Modular/ControllerRevB/Controller.kicad_pcb (KiCad board)
At the start: 2 copper layers, 55.2 x 33 mm, 19 parts, among them J1 Barrel_Jack, J2 Conn_01x05, J3 Conn_02x08_Odd_Even, J4 Conn_02x04_Odd_Even, SW1 SW_SPST, SW2 Rotary_Encoder, SW3 SW_SPST, U1 STM32F051K8Tx, U2 L78L33_SOT89

Commit message: hw update
controller revb
Parts:
- removed R1: 10K, Resistor_SMD:R_1206_3216Metric_Pad1.42x1.75mm_HandSolder
- added BZ1: Buzzer, Connector_PinHeader_2.54mm:PinHeader_1x02_P2.54mm_Vertical, B.Cu at (124.6, 117.6)
- added D1: D, Diode_SMD:D_SOD-123F, F.Cu at (124.1, 120.9)
- added Q1: MMBT3904, Package_TO_SOT_SMD:SOT-23, F.Cu at (128.4, 115.1)
- added SW4: SW_SPST, Connector_PinHeader_2.54mm:PinHeader_1x02_P2.54mm_Vertical, B.Cu at (146.3, 123.1)
- added U3: MCP1416, Package_TO_SOT_SMD:SOT-23-5, F.Cu at (132.8, 115.1)
- SW1, SW3: moved to B.Cu
- moved R4 11.4 mm to (133.3, 120.9), turned to 180 degrees
- moved SW1 11.1 mm to (139.6, 123.1), turned to 0 degrees
- moved SW3 10.2 mm to (151.3, 123.1), turned to 0 degrees
- moved J4 7.62 mm to (154.4, 106.2)
- moved U1 7.62 mm to (143.4, 112.6)
Connections:
- net /LED_Controller_Module/MINUTE_BTN renamed /LED_Controller_Module/UP_BTN
- U1 pad 27: Net-(U1-Pad27) -> /LED_Controller_Module/BUZZER_PWM
- U1 pad 7: Net-(U1-Pad7) -> /LED_Controller_Module/DOWN_BTN
Routing:
- net VPP: track 81.1 -> 126.8 mm
- net Net-(BZ1-Pad2): track 0.00 -> 10.7 mm
- net /LED_Controller_Module/SWCLK: track 21.9 -> 29.7 mm
- net /LED_Controller_Module/SWDIO: track 17.4 -> 25.1 mm
- net /LED_Controller_Module/ENC_A: track 6.49 -> 14.0 mm
- net /LED_PWM_OUT5: track 14.7 -> 22.1 mm
- net /LED_PWM_OUT1: track 22.4 -> 29.7 mm
- net /LED_Controller_Module/BUZZER_PWM: track 0.00 -> 7.19 mm
- net /LED_Controller_Module/ENC_B: track 9.64 -> 16.7 mm
- net /LED_PWM_OUT2: track 15.3 -> 22.3 mm
- net /LED_PWM_OUT3: track 10.5 -> 17.2 mm
- net /LED_PWM_OUT4: track 9.81 -> 16.1 mm
- net GNDS: track 63.8 -> 69.3 mm, vias 8 -> 9
- net /LED_Controller_Module/NRST: track 34.9 -> 39.1 mm
- net /LED_Controller_Module/DOWN_BTN: track 0.00 -> 4.09 mm
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
Commit message: updated
Parts:
- added R1: 1K, Resistor_SMD:R_1206_3216Metric_Pad1.42x1.75mm_HandSolder, F.Cu at (136.1, 114.6)
- J1: footprint Connector_Molex:Molex_KK-396_A-41791-0002_1x02_P3.96mm_Vertical -> Connector_Molex:Molex_KK-254_AE-6410-02A_1x02_P2.54mm_Vertical
- R4: value 0R -> 1K
- moved D1 6.42 mm to (124.3, 114.5), turned to 270 degrees
- moved SW1 5.84 mm to (145.4, 123.2)
- moved BZ1 5.41 mm to (127.6, 113.1), turned to 180 degrees
- moved Q1 5.31 mm to (125.2, 119.3)
- moved U3 4.77 mm to (135.0, 119.3)
- moved R4 3.42 mm to (130.0, 120.3), turned to 0 degrees
- moved J1 2.36 mm to (109.5, 107.6), turned to 270 degrees
- moved SW4 1.66 mm to (148.0, 123.2)
- moved SW3 0.77 mm to (150.5, 123.2)
Connections:
- R4 pad 1: Net-(R1-Pad2) -> Net-(Q1-Pad1)
- R4 pad 2: GNDS -> Net-(R4-Pad2)
- U1 pad 31: Net-(R1-Pad2) -> GNDS
- U3 pad 3: /LED_Controller_Module/BUZZER_PWM -> Net-(R1-Pad1)
- U3 pad 5: Net-(Q1-Pad1) -> Net-(R4-Pad2)
Routing:
- net VPP: track 126.8 -> 157.4 mm, vias 0 -> 2
- net Net-(R1-Pad2): track 8.94 -> 0.00 mm
- net Net-(BZ1-Pad2): track 10.7 -> 6.84 mm
- net /LED_Controller_Module/ENABLE_LED: track 4.44 -> 7.84 mm
- net /LED_Controller_Module/NRST: track 39.1 -> 36.0 mm
- net /LED_Controller_Module/BUZZER_PWM: track 7.19 -> 4.54 mm
- net Net-(R4-Pad2): track 0.00 -> 2.43 mm
- net +3V3: track 91.2 -> 88.8 mm
- net Net-(R1-Pad1): track 0.00 -> 2.33 mm
- net /LED_Controller_Module/DOWN_BTN: track 4.09 -> 4.90 mm
- net GNDS: track 69.3 -> 68.7 mm, vias 9 -> 8
