File: UV_LED_Driver_Modular/ControllerRevB/RotaryEncoderNoSwitch.sch (KiCad schematic (older format))
At the start: 3 parts, among them SW2 Rotary_Encoder

Commit message: Updated prototype designs for fab
updated readme
Parts:
- R2, R3: footprint Resistor_SMD:R_1206_3216Metric_Pad1.42x1.75mm_HandSolder -> Resistor_SMD:R_0805_2012Metric_Pad1.15x1.40mm_HandSolder
Changed lines of the file:
@@
 $Descr A4 11693 8268
 encoding utf-8
-Sheet 3 3
+Sheet 3 4
 Title ""
 Date ""
@@
 F 0 "R2" H 5445 4196 50  0000 L CNN
 F 1 "10K" H 5445 4105 50  0000 L CNN
-F 2 "Resistor_SMD:R_1206_3216Metric_Pad1.42x1.75mm_HandSolder" V 5305 4150 50  0001 C CNN
+F 2 "Resistor_SMD:R_0805_2012Metric_Pad1.15x1.40mm_HandSolder" V 5305 4150 50  0001 C CNN
 F 3 "~" H 5375 4150 50  0001 C CNN
 	1    5375 4150
@@
 F 0 "R3" H 6620 4196 50  0000 L CNN
 F 1 "10K" H 6620 4105 50  0000 L CNN
-F 2 "Resistor_SMD:R_1206_3216Metric_Pad1.42x1.75mm_HandSolder" V 6480 4150 50  0001 C CNN
+F 2 "Resistor_SMD:R_0805_2012Metric_Pad1.15x1.40mm_HandSolder" V 6480 4150 50  0001 C CNN
 F 3 "~" H 6550 4150 50  0001 C CNN
 	1    6550 4150
