File: UV_LED_Driver_Modular/ControllerRevB/LED_Controller.sch (KiCad schematic (older format))
At the start: 19 parts, among them J1 Barrel_Jack, J2 Conn_01x05, J4 Conn_02x04_Odd_Even, J5 Conn_01x01, J6 Conn_01x01, Q1 MMBT3904, SW1 SW_SPST, SW3 SW_SPST, SW4 SW_SPST, U1 STM32F051K8Tx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

Commit message: added pull down resistor to MCU to prevent buzzer from sounding at boot
Parts:
- R1: value 1K -> 10K
Connections:
- net BUZZER_PWM: now also U3.3 (IN)
- net GNDS: now also R1.1
Other:
- moved on the sheet: R1
Changed lines of the file:
@@
 Text Label 7350 5300 0    50   ~ 0
 BUZZER_PWM
-Wire Wire Line
-	7350 5300 8000 5300
 $Comp
 L Switch:SW_SPST SW4
@@
 L Device:R R1
 U 1 1 5EF88709
-P 8150 5300
-F 0 "R1" V 7943 5300 50  0000 C CNN
-F 1 "1K" V 8034 5300 50  0000 C CNN
-F 2 "Resistor_SMD:R_0805_2012Metric_Pad1.15x1.40mm_HandSolder" V 8080 5300 50  0001 C CNN
-F 3 "~" H 8150 5300 50  0001 C CNN
-	1    8150 5300
-	0    1    1    0
-$EndComp
-Wire Wire Line
-	8300 5300 8500 5300
+P 8150 5550
+F 0 "R1" H 8300 5500 50  0000 C CNN
+F 1 "10K" H 8300 5600 50  0000 C CNN
+F 2 "Resistor_SMD:R_0805_2012Metric_Pad1.15x1.40mm_HandSolder" V 8080 5550 50  0001 C CNN
+F 3 "~" H 8150 5550 50  0001 C CNN
+	1    8150 5550
+	-1   0    0    1
+$EndComp
 $Comp
 L Device:R R4
@@
 Wire Wire Line
 	10200 3875 10200 4125
+Wire Wire Line
+	7350 5300 8150 5300
+Wire Wire Line
+	8150 5400 8150 5300
+Connection ~ 8150 5300
+Wire Wire Line
+	8150 5300 8500 5300
+$Comp
+L power:GNDS #PWR?
+U 1 1 5F04EE6A
+P 8150 5800
+F 0 "#PWR?" H 8150 5550 50  0001 C CNN
+F 1 "GNDS" H 8155 5627 50  0000 C CNN
+F 2 "" H 8150 5800 50  0001 C CNN
+F 3 "" H 8150 5800 50  0001 C CNN
+	1    8150 5800
+	-1   0    0    -1
+$EndComp
+Wire Wire Line
+	8150 5800 8150 5700
 $EndSCHEMATC
